Commit message: commit from robot

File: panda_table_description/urdf/panda_table.urdf.xacro (robot description, xacro)
@@ -102,17 +102,17 @@
     </collision>
    </link>
-   <link name="work_piece">
-    <visual>
-      <geometry>
-	<mesh filename="package://panda_table_description/meshes/work_piece.stl" scale="0.001 0.001 0.001"/>
-      </geometry>
-      <origin rpy="0 1.5707 0" xyz="0.0 0.0 0.0" />
-    </visual>
-    <collision>
-      <geometry>
-	<mesh filename="package://panda_table_description/meshes/work_piece.stl" scale="0.001 0.001 0.001"/>
-      </geometry>
-      <origin rpy="0 1.5707 0" xyz="0.0 0.0 0.0" />
-    </collision>
+   <link name="camera_link">
+     <inertial>
+       <mass value="0.01"/>
+       <inertia ixx="0.001" ixy="0" ixz="0" iyy="0.001" iyz="0" izz="0.001" />
+       <origin/>
+     </inertial>
+     <visual>
+       <origin xyz="0 0 0" rpy="0 0 0" />
+       <geometry>
+         <box size="0.05 0.05 0.005" />
+       </geometry>
+       <material name="orange"/>
+     </visual>
    </link>
   <joint name="world_joint" type="fixed">
@@ -124,5 +124,5 @@
     <parent link="table" />
     <child link = "mount_flange_link" />
-    <origin xyz="0.0 0.425 0.7" rpy="0.0 0.0 1.5707" />
+    <origin xyz="0.0 0.305 0.7" rpy="0.0 0.0 1.5707" />
   </joint>
   <joint name="table_column1" type="fixed">
@@ -136,8 +136,8 @@
     <origin xyz="-0.45 -0.505 0.7" rpy="0.0 0.0 0.0" />
   </joint>
-  <joint name="table_wp" type="fixed">
-    <parent link="table" />
-    <child link = "work_piece" />
-    <origin xyz="0.45 0.105 0.72" rpy="0.0 0.0 0.0" />
+  <joint name="world_camera_joint" type="fixed">
+    <parent link="world" />
+    <child link = "camera_link" />
+    <origin xyz="-0.045 -0.85 1.31" rpy="0.0 0.745 1.56" />
   </joint>
 </robot>
